Commit message: saving sensor values

File: body.urdf (robot description, URDF)
Before this commit: robot robot, 3 links, 2 joints
Joints:
- removed joint BackLeg_Torso
- removed joint Torso_FrontLeg
- added joint FrontLeg_Torso: type revolute, parent FrontLeg, child Torso, origin xyz=0.0 0.5 1.0 rpy=0 0 0, axis 0 1 0, limit lower=-3.14159 upper=3.14159 effort=0.0 velocity=0.0
- added joint Torso_BackLeg: type revolute, parent Torso, child BackLeg, origin xyz=0.0 0.5 -0.5 rpy=0 0 0, axis 0 1 0, limit lower=-3.14159 upper=3.14159 effort=0.0 velocity=0.0

Commit message: F. sensors

File: body.urdf (robot description, URDF)
Before this commit: robot robot, 3 links, 2 joints
Joints:
- removed joint FrontLeg_Torso
- added joint Torso_FrontLeg: type revolute, parent Torso, child FrontLeg, origin xyz=0.0 0.5 1.0 rpy=0 0 0, axis 0 1 0, limit lower=-3.14159 upper=3.14159 effort=0.0 velocity=0.0
- joint Torso_BackLeg: origin xyz=0.0 0.5 -0.5 rpy=0 0 0 -> xyz=0.0 -0.5 1.0 rpy=0 0 0

Commit message: G. move forward with motors

File: body.urdf (robot description, URDF)
Before this commit: robot robot, 3 links, 2 joints
Joints:
- joint Torso_BackLeg: origin xyz=0.0 -0.5 1.0 rpy=0 0 0 -> xyz=0.5 0 1.0 rpy=0 0 0
- joint Torso_FrontLeg: origin xyz=0.0 0.5 1.0 rpy=0 0 0 -> xyz=-0.5 0 1.0 rpy=0 0 0

Commit message: N. changed joint axes

File: body.urdf (robot description, URDF)
Before this commit: robot robot, 3 links, 2 joints
Links:
- link BackLeg: geometry collision box size=0.2 1.0 0.2; visual box size=0.2 1.0 0.2
- link FrontLeg: geometry collision box size=0.2 1.0 0.2; visual box size=0.2 1.0 0.2
Joints:
- joint Torso_BackLeg: axis 0 1 0 -> 1 0 0; origin xyz=0.5 0 1.0 rpy=0 0 0 -> xyz=0.0 -0.5 1.0 rpy=0 0 0
- joint Torso_FrontLeg: axis 0 1 0 -> 1 0 0; origin xyz=-0.5 0 1.0 rpy=0 0 0 -> xyz=0.0 0.5 1.0 rpy=0 0 0
